File: PHONE.sch (EAGLE design)
At the start: 105 parts, among them IC1 ATMEGA1284P, IC2 ATMEGA16U2-MU, IC3 LTC4054, IC5 LP2985-33DBVR, J1 Power, J2 Analog, J3 Digital_8_13, J4 Digital_0_7, P1 USB-6PSMT, P2 ICSP:MAIN, P3 ICSP:USB, Q1 2N7002 SOT-23, Q2 2N7002, Q3 BC846ALTIG, SW0 0, SW1 1, SW10 *, SW11 #, SW12 LEFT, SW13 DOWN, SW14 RIGHT, SW15 UP, SW2 2, SW3 3, SW4 4, SW5 5, SW6 6, SW7 7, SW8 8, SW9 9, X1 8MHz, X2 16MHz

Commit message: v1.0 release
Parts:
- removed C14: 100nF 0603, freetronics:CAP0603
- removed P3: ICSP:USB, pinhead:PINHD-2X3
- removed R20, R21: 10K 0603, freetronics:RESISTOR0603
- removed R22: 1K 0603, freetronics:RESISTOR0603
- removed X2: 16MHz, freetronics-master-v1:CRYSTALHC49UV
- removed Z1, Z2: PGB1010603, freetronics:RESISTOR0603
- added C10: 33pF 0603, freetronics:CAP0603
- added C11: 100nF 0603, freetronics:CAP0603
- added JP11: M01PTH, freetronics-original:M01PTH
- added JP12: MIC, freetronics-master-v1.1:M02PTH
- added JP13: SPKR, freetronics-master-v1.1:M02PTH
- added JP14: PIEZO, freetronics-master-v1.1:M02PTH
- added TP3, TP4, TP5: TEST-POINT, freetronics-original:TEST-POINT2
- C12, C13: value 22pF 0603 -> 47pF 0603; device freetronics:CAP0603 -> freetronics-jon:C-EUC0603
- C5: value 47uF 25V -> 100uF 16V
- C6: value 1uF 0603 -> 100uF 16V; device freetronics:CAP0603 -> rcl:CPOL-EUD
- IC2: value ATMEGA16U2-MU -> FT230X; device freetronics-jon:ATMEL_ATMEGA8U2-MUQFN -> freetronics-jon:FT230X
- R11: value 10K 0603 -> 27R 0603
- R12: value 1M 0603 -> 27R 0603
- R13: value 27R 0603 -> 1K 0603
- R14, R15: value 22R 0603 -> 10K 0603
- R16: value 1K 0603 -> 3K3 0603
- R19: value 3K3 0603 -> 1K 0603
- SJ2: value GROUND -> (none); device freetronics-jon:SJCN -> freetronics-master-v1.1:SJ
- SJ3: value UBOOT -> (none); device jumper:SJ -> freetronics-master-v1.1:SJ
- renumbered IC5 to IC4
Connections:
- removed net MISO2: IC2.(MISO)PB3, P3.1
- removed net MOSI2: IC2.(MOSI)PB2, P3.4
- removed net N$113: C12.2, IC2.XTAL2, R12.2, X2.2
- removed net N$114: C13.2, R12.1, R13.2, X2.1
- removed net N$117: C6.1, IC2.UCAP
- removed net RESET2: IC2.RESET, P3.5, R11.1
- removed net SCK2: IC2.(SCLK)PB1, P3.3
- removed net UGND: IC2.UGND, L1.2, P1.GND, SJ2.1
- removed net USBVCC: C1.2, F1.2, IC2.UVCC, IC3.VCC, R16.1, R17.1
- removed net VIN: J1.8
- new net N$27: JP12.1, SJ2.1
- new net N$28: JP12.2, SJ3.1
- net 5V: now also C1.2, F1.2, IC3.VCC, R13.1, R14.1; no longer C14.1, IC2.AVCC, P3.2, R11.2
- net D9: now also JP14.1
- net DTR: now also IC2.!RTS; no longer IC2.(CTS)PD7, SJ3.2
- net GND: now also C10.1, C11.2, C6.-, IC2.GND@13, IC2.GND@17, IC2.GND@3, JP11.1, JP14.2, L1.2, P1.GND, R15.2, R16.2, R17.2, R19.1; no longer C12.1, C13.1, C14.2, C6.2, IC2.GND, IC2.PAD, P3.6, R18.2, R19.2, R20.2, R22.1, SJ2.2, SJ3.1
- net N$10: now also R14.2; no longer R17.2
- net N$12: now also R15.1; no longer R18.1
- net N$15: now also R18.1; no longer R21.1
- net N$16: now also C12.1, R12.2; no longer R15.2, Z1.1
- net N$17: now also C13.1, R11.2; no longer R14.2, Z2.1
- net N$18: now also SJ3.2
- net N$19: now also JP13.2
- net N$2: now also C11.1, IC2.!RESET, IC2.3V3OUT, IC2.VCCIO; no longer IC2.XTAL1, R13.1
- net N$20: now also JP13.1
- net N$23: now also TP3.1
- net N$24: now also TP4.1
- net N$25: now also TP5.1
- net N$26: now also R18.2; no longer R21.2
- net N$3: now also C12.2, C13.2; no longer Z1.2, Z2.2
- net N$33: now also R16.1; no longer R19.1
- net N$34: now also R17.1; no longer R20.1
- net N$7: now also R19.2; no longer R22.2
- net N$8: now also R13.2; no longer R16.2
- net N$9: now also SJ2.2
- net RD+: now also IC2.USBDP, R12.1; no longer IC2.D+, R15.1
- net RD-: now also IC2.USBDM, R11.1; no longer IC2.D-, R14.1
- net RXLED: now also IC2.CBUS2; no longer IC2.PD4
- net TXLED: now also IC2.CBUS1; no longer IC2.(XCK)PD5
- net USBRXD: now also IC2.TXD; no longer IC2.(TXD1)PD3
- net USBTXD: now also IC2.RXD; no longer IC2.(RXD1)PD2
- net VCC: now also C10.2, C6.+, J1.8
Other:
- note added: "ICSP Header"
- note added: "PIEZO"
- note removed: "(Linked)"
- note removed: "ATmega16U2 Microcontroller"
- note removed: "ICSP Headers"
- moved on the sheet: C12, C13, F1, L1, LED1, LED2, LED7, P1, R11, R12, R13, R14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

Commit message: v1.1 release: separated AUDIO_GND from system GND
Parts:
- R10: value 1K5 0603 -> 820R 0603
- R14: value 10K 0603 -> 1K 0603
- R19: value 1K 0603 -> 2K7 0603
- SJ6: device freetronics-jon:SJCN -> freetronics-master-v1.1:SJ
Connections:
- removed net D7: IC1.PD7(OC2A/PCINT31), J4.8
- removed net N$28: JP12.2, SJ3.1
- removed net OLED_DNC: JP1.9
- new net AUDIO_GND: JP12.2, S5.GND@42, SJ3.1
- new net D7_OLED_DNC: IC1.PD7(OC2A/PCINT31), J4.8, JP1.9
- net GND: no longer S5.GND@42
Other:
- note added: "V1.1 (2013-11-26)"
- note removed: "V1.0 (2013-10-28)"
- moved on the sheet: SJ2, SJ3
Changed lines of the file:
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@@
 <part name="P2" library="pinhead" deviceset="PINHD-2X3" device="" value="ICSP:MAIN"/>
 <part name="GND22" library="SparkFun" deviceset="GND" device=""/>
-<part name="R10" library="freetronics" deviceset="RESISTOR" device="0603" value="1K5 0603"/>
+<part name="R10" library="freetronics" deviceset="RESISTOR" device="0603" value="820R 0603"/>
 <part name="LED4" library="freetronics-master-v1" deviceset="LED" device="0603" value="3V3/BLUE"/>
 <part name="GND23" library="SparkFun" deviceset="GND" device=""/>
@@
 <part name="S5" library="freetronics-jon" deviceset="ADH8066" device="" value="Hirose DF12C(3.0)-50DP-0.5V"/>
 <part name="GND12" library="SparkFun" deviceset="GND" device=""/>
-<part name="GND13" library="SparkFun" deviceset="GND" device=""/>
 <part name="JP1" library="freetronics-original" deviceset="M05X2" device="PTH"/>
 <part name="GND15" library="SparkFun" deviceset="GND" device=""/>
@@
 <part name="IC3" library="freetronics-luke" deviceset="LTC4054" device=""/>
 <part name="R13" library="freetronics" deviceset="RESISTOR" device="0603" value="1K 0603"/>
-<part name="R14" library="freetronics" deviceset="RESISTOR" device="0603" value="10K 0603"/>
+<part name="R14" library="freetronics" deviceset="RESISTOR" device="0603" value="1K 0603"/>
 <part name="C1" library="freetronics" deviceset="CAP" device="0603" value="1uF 0603"/>
 <part name="R15" library="freetronics" deviceset="RESISTOR" device="0603" value="10K 0603"/>
@@
 <part name="LED7" library="freetronics-master-v1" deviceset="LED" device="0603" value="5V/JADEGREEN"/>
 <part name="GND14" library="SparkFun" deviceset="GND" device=""/>
-<part name="R19" library="freetronics" deviceset="RESISTOR" device="0603" value="1K 0603"/>
+<part name="R19" library="freetronics" deviceset="RESISTOR" device="0603" value="2K7 0603"/>
 <part name="U$3" library="SparkFun" deviceset="5V" device=""/>
-<part name="SJ6" library="freetronics-jon" deviceset="SJC" device="N" value="LINK"/>
+<part name="SJ6" library="freetronics-master-v1.1" deviceset="SJ" device="" value="LINK"/>
 <part name="U$6" library="freetronics" deviceset="FIDUCIAL" device="1X2.5"/>
 <part name="U$7" library="freetronics" deviceset="FIDUCIAL" device="1X2.5"/>
@@
 <frame x1="0" y1="0" x2="248.92" y2="185.42" columns="8" rows="5" layer="94"/>
 <text x="7.62" y="175.26" size="3.048" layer="94">ArduPhone</text>
-<text x="7.62" y="169.418" size="1.778" layer="94">V1.0 (2013-10-28)</text>
+<text x="7.62" y="169.418" size="1.778" layer="94">V1.1 (2013-11-26)</text>
 <text x="53.34" y="164.338" size="1.778" layer="94">SKU: PHONE</text>
 <text x="7.366" y="164.338" size="1.778" layer="94">(C)2013 Freetronics Pty Ltd</text>
@@
 <text x="73.66" y="20.32" size="1.778" layer="97">OLED_CS</text>
 <text x="73.66" y="25.4" size="1.778" layer="97">SD_CS</text>
-<text x="157.48" y="167.64" size="1.778" layer="94">TODO:
+<text x="149.86" y="160.02" size="1.778" layer="94">TODO:
 Antenna mount
 Power switch</text>
@@
 <instance part="S5" gate="G$1" x="71.12" y="238.76"/>
 <instance part="GND12" gate="1" x="43.18" y="203.2"/>
-<instance part="GND13" gate="1" x="129.54" y="246.38"/>
 <instance part="JP1" gate="G$1" x="53.34" y="137.16"/>
 <instance part="GND15" gate="1" x="66.04" y="142.24" rot="R90"/>
@@
 </instance>
 <instance part="U$3" gate="G$1" x="78.74" y="111.76"/>
-<instance part="SJ6" gate="G$1" x="104.14" y="259.08" smashed="yes" rot="R270">
-<attribute name="NAME" x="106.68" y="259.08" size="1.778" layer="95"/>
-<attribute name="VALUE" x="106.68" y="256.794" size="1.778" layer="96"/>
+<instance part="SJ6" gate="1" x="99.06" y="259.08" smashed="yes" rot="R270">
+<attribute name="NAME" x="101.6" y="259.08" size="1.778" layer="95"/>
+<attribute name="VALUE" x="101.6" y="256.794" size="1.778" layer="96"/>
 </instance>
 <instance part="U$6" gate="G$1" x="88.9" y="177.8"/>
@@
 <instance part="GND17" gate="1" x="177.8" y="203.2"/>
 <instance part="JP12" gate="G$1" x="149.86" y="251.46" rot="MR0"/>
-<instance part="SJ2" gate="1" x="134.62" y="251.46" smashed="yes" rot="R180">
-<attribute name="NAME" x="134.62" y="254" size="1.27" layer="95" rot="R90"/>
-</instance>
-<instance part="SJ3" gate="1" x="129.54" y="254" smashed="yes" rot="R180">
-<attribute name="NAME" x="129.54" y="256.54" size="1.27" layer="95" rot="R90"/>
+<instance part="SJ2" gate="1" x="129.54" y="251.46" smashed="yes" rot="R180">
+<attribute name="NAME" x="129.54" y="254" size="1.27" layer="95" rot="R90"/>
+</instance>
+<instance part="SJ3" gate="1" x="111.76" y="254" smashed="yes" rot="R180">
+<attribute name="NAME" x="111.76" y="256.54" size="1.27" layer="95" rot="R90"/>
 </instance>
 <instance part="JP13" gate="G$1" x="149.86" y="276.86" rot="MR0"/>
@@
 <wire x1="43.18" y1="256.54" x2="43.18" y2="218.44" width="0.1524" layer="91"/>
 <junction x="43.18" y="218.44"/>
-</segment>
-<segment>
-<pinref part="S5" gate="G$1" pin="GND@42"/>
-<pinref part="GND13" gate="1" pin="GND"/>
-<wire x1="93.98" y1="248.92" x2="129.54" y2="248.92" width="0.1524" layer="91"/>
 </segment>
 <segment>
@@
 </segment>
 </net>
-<net name="D7" class="0">
+<net name="D7_OLED_DNC" class="0">
 <segment>
 <wire x1="48.26" y1="27.94" x2="60.96" y2="27.94" width="0.1524" layer="91"/>
@@
 <wire x1="195.58" y1="7.62" x2="208.28" y2="7.62" width="0.1524" layer="91"/>
 <label x="198.12" y="7.62" size="1.778" layer="95"/>
+</segment>
+<segment>
+<pinref part="JP1" gate="G$1" pin="9"/>
+<wire x1="45.72" y1="132.08" x2="27.94" y2="132.08" width="0.1524" layer="91"/>
+<label x="30.48" y="132.08" size="1.778" layer="95"/>
 </segment>
 </net>
@@
 <pinref part="S5" gate="G$1" pin="EARN"/>
 <pinref part="S4" gate="G$1" pin="1"/>
-<wire x1="93.98" y1="269.24" x2="104.14" y2="269.24" width="0.1524" layer="91"/>
-<pinref part="SJ6" gate="G$1" pin="1"/>
-<wire x1="104.14" y1="269.24" x2="116.84" y2="269.24" width="0.1524" layer="91"/>
+<wire x1="93.98" y1="269.24" x2="99.06" y2="269.24" width="0.1524" layer="91"/>
+<pinref part="SJ6" gate="1" pin="1"/>
+<wire x1="99.06" y1="269.24" x2="116.84" y2="269.24" width="0.1524" layer="91"/>
 <wire x1="116.84" y1="269.24" x2="121.92" y2="269.24" width="0.1524" layer="91"/>
-<wire x1="104.14" y1="264.16" x2="104.14" y2="269.24" width="0.1524" layer="91"/>
-<junction x="104.14" y="269.24"/>
+<wire x1="99.06" y1="264.16" x2="99.06" y2="269.24" width="0.1524" layer="91"/>
+<junction x="99.06" y="269.24"/>
 <wire x1="116.84" y1="279.4" x2="116.84" y2="269.24" width="0.1524" layer="91"/>
 <junction x="116.84" y="269.24"/>
@@
 <wire x1="195.58" y1="38.1" x2="208.28" y2="38.1" width="0.1524" layer="91"/>
 <label x="198.12" y="38.1" size="1.778" layer="95"/>
-</segment>
-</net>
-<net name="OLED_DNC" class="0">
-<segment>
-<pinref part="JP1" gate="G$1" pin="9"/>
-<wire x1="45.72" y1="132.08" x2="27.94" y2="132.08" width="0.1524" layer="91"/>
-<label x="30.48" y="132.08" size="1.778" layer="95"/>
 </segment>
 </net>
@@
 <junction x="119.38" y="259.08"/>
 <pinref part="SJ2" gate="1" pin="2"/>
-<wire x1="129.54" y1="251.46" x2="119.38" y2="251.46" width="0.1524" layer="91"/>
+<wire x1="124.46" y1="251.46" x2="119.38" y2="251.46" width="0.1524" layer="91"/>
 <junction x="119.38" y="251.46"/>
 </segment>
@@
 <segment>
 <pinref part="S5" gate="G$1" pin="MIC1_N"/>
-<wire x1="93.98" y1="254" x2="104.14" y2="254" width="0.1524" layer="91"/>
-<pinref part="SJ6" gate="G$1" pin="2"/>
+<wire x1="93.98" y1="254" x2="99.06" y2="254" width="0.1524" layer="91"/>
+<pinref part="SJ6" gate="1" pin="2"/>
 <pinref part="SJ3" gate="1" pin="2"/>
-<wire x1="124.46" y1="254" x2="104.14" y2="254" width="0.1524" layer="91"/>
-<junction x="104.14" y="254"/>
+<wire x1="106.68" y1="254" x2="99.06" y2="254" width="0.1524" layer="91"/>
+<junction x="99.06" y="254"/>
 </segment>
 </net>
@@
 <pinref part="SJ2" gate="1" pin="1"/>
 <pinref part="JP12" gate="G$1" pin="1"/>
-<wire x1="142.24" y1="251.46" x2="139.7" y2="251.46" width="0.1524" layer="91"/>
-</segment>
-</net>
-<net name="N$28" class="0">
-<segment>
+<wire x1="142.24" y1="251.46" x2="134.62" y2="251.46" width="0.1524" layer="91"/>
+</segment>
+</net>
+<net name="AUDIO_GND" class="0">
+<segment>
+<pinref part="S5" gate="G$1" pin="GND@42"/>
+<wire x1="93.98" y1="248.92" x2="121.92" y2="248.92" width="0.1524" layer="91"/>
 <pinref part="SJ3" gate="1" pin="1"/>
 <pinref part="JP12" gate="G$1" pin="2"/>
-<wire x1="134.62" y1="254" x2="142.24" y2="254" width="0.1524" layer="91"/>
-</segment>
-</net>
+<wire x1="116.84" y1="254" x2="121.92" y2="254" width="0.1524" layer="91"/>
+<wire x1="121.92" y1="254" x2="142.24" y2="254" width="0.1524" layer="91"/>
+<wire x1="121.92" y1="248.92" x2="121.92" y2="254" width="0.1524" layer="91"/>
+<junction x="121.92" y="254"/>
+<label x="96.52" y="248.92" size="1.778" layer="95"/>
+</segment>
+</net>

Commit message: Switched to 4 layers and rerouted for v1.2 release
Parts:
- SJ2: value (none) -> SJCN; device freetronics-master-v1.1:SJ -> freetronics-jon:SJCN
Other:
- note added: "V1.2 (2013-11-26)"
- note removed: "V1.1 (2013-11-26)"
Changed lines of the file:
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@@
 <part name="GND17" library="SparkFun" deviceset="GND" device=""/>
 <part name="JP12" library="freetronics-master-v1.1" deviceset="M02" device="PTH" value="MIC"/>
-<part name="SJ2" library="freetronics-master-v1.1" deviceset="SJ" device=""/>
+<part name="SJ2" library="freetronics-jon" deviceset="SJC" device="N"/>
 <part name="SJ3" library="freetronics-master-v1.1" deviceset="SJ" device=""/>
 <part name="JP13" library="freetronics-master-v1.1" deviceset="M02" device="PTH" value="SPKR"/>
@@
 <frame x1="0" y1="0" x2="248.92" y2="185.42" columns="8" rows="5" layer="94"/>
 <text x="7.62" y="175.26" size="3.048" layer="94">ArduPhone</text>
-<text x="7.62" y="169.418" size="1.778" layer="94">V1.1 (2013-11-26)</text>
+<text x="7.62" y="169.418" size="1.778" layer="94">V1.2 (2013-11-26)</text>
 <text x="53.34" y="164.338" size="1.778" layer="94">SKU: PHONE</text>
 <text x="7.366" y="164.338" size="1.778" layer="94">(C)2013 Freetronics Pty Ltd</text>
@@
 <text x="73.66" y="20.32" size="1.778" layer="97">OLED_CS</text>
 <text x="73.66" y="25.4" size="1.778" layer="97">SD_CS</text>
-<text x="149.86" y="160.02" size="1.778" layer="94">TODO:
+<text x="149.86" y="167.64" size="1.778" layer="94">TODO:
 Antenna mount
 Power switch</text>
@@
 <text x="10.16" y="271.78" size="1.778" layer="94" ratio="12">GSM Module</text>
 <text x="7.62" y="149.86" size="1.778" layer="94" ratio="12">LCD Module Header</text>
-<text x="114.3" y="177.8" size="1.778" layer="94" ratio="12">USB-Serial Converter</text>
+<text x="106.68" y="177.8" size="1.778" layer="94" ratio="12">USB-Serial Converter</text>
 <text x="228.6" y="360.68" size="1.6764" layer="94" ratio="12">Output</text>
 <text x="172.72" y="360.68" size="1.6764" layer="94" ratio="12">Input</text>
@@
 <instance part="GND17" gate="1" x="177.8" y="203.2"/>
 <instance part="JP12" gate="G$1" x="149.86" y="251.46" rot="MR0"/>
-<instance part="SJ2" gate="1" x="129.54" y="251.46" smashed="yes" rot="R180">
+<instance part="SJ2" gate="G$1" x="129.54" y="251.46" smashed="yes" rot="R180">
 <attribute name="NAME" x="129.54" y="254" size="1.27" layer="95" rot="R90"/>
 </instance>
@@
 <wire x1="119.38" y1="251.46" x2="119.38" y2="259.08" width="0.1524" layer="91"/>
 <junction x="119.38" y="259.08"/>
-<pinref part="SJ2" gate="1" pin="2"/>
+<pinref part="SJ2" gate="G$1" pin="2"/>
 <wire x1="124.46" y1="251.46" x2="119.38" y2="251.46" width="0.1524" layer="91"/>
 <junction x="119.38" y="251.46"/>
@@
 <net name="N$27" class="0">
 <segment>
-<pinref part="SJ2" gate="1" pin="1"/>
+<pinref part="SJ2" gate="G$1" pin="1"/>
 <pinref part="JP12" gate="G$1" pin="1"/>
 <wire x1="142.24" y1="251.46" x2="134.62" y2="251.46" width="0.1524" layer="91"/>
