File: PHONE.sch (EAGLE design)
At the start: 106 parts, among them IC1 ATMEGA1284P, IC2 FT230X, IC3 LTC4054, IC4 LP2985-33DBVR, J1 Power, J2 Analog, J3 Digital_8_13, J4 Digital_0_7, P1 USB-6PSMT, P2 ICSP:MAIN, Q1 2N7002 SOT-23, Q2 2N7002, Q3 BC846ALTIG, SW0 0, SW1 1, SW10 *, SW11 #, SW12 LEFT, SW13 DOWN, SW14 RIGHT, SW15 UP, SW2 2, SW3 3, SW4 4, SW5 5, SW6 6, SW7 7, SW8 8, SW9 9, X1 8MHz

Commit message: Reconciled schematic and layout using common parts
Parts:
- C1, C11, C2, C3, C4, C7, C8, C9: device freetronics:CAP0603 -> freetronics-master-v1.1:CAP0603
- R1, R10, R11, R12, R13, R14, R15, R16, R17, R18, R19, R2, R3, R4, R5, R6, R7, R8, R9: device freetronics:RESISTOR0603 -> freetronics-master-v1.1:RESISTOR0603
Changed lines of the file:
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@@
 <?xml version="1.0" encoding="utf-8"?>
 <!DOCTYPE eagle SYSTEM "eagle.dtd">
-<eagle version="6.3">
+<eagle version="6.5.0">
 <drawing>
 <settings>
@@
 <part name="J4" library="freetronics" deviceset="M08" device="" value="Digital_0_7"/>
 <part name="X1" library="freetronics-master-v1" deviceset="CRYSTAL" device="HC49UV" value="8MHz"/>
-<part name="C2" library="freetronics" deviceset="CAP" device="0603" value="22pF 0603"/>
-<part name="C3" library="freetronics" deviceset="CAP" device="0603" value="22pF 0603"/>
+<part name="C2" library="freetronics-master-v1.1" deviceset="CAP" device="0603" value="22pF 0603"/>
+<part name="C3" library="freetronics-master-v1.1" deviceset="CAP" device="0603" value="22pF 0603"/>
 <part name="GND2" library="SparkFun" deviceset="GND" device=""/>
-<part name="C4" library="freetronics" deviceset="CAP" device="0603" value="100nF 0603"/>
+<part name="C4" library="freetronics-master-v1.1" deviceset="CAP" device="0603" value="100nF 0603"/>
 <part name="GND3" library="SparkFun" deviceset="GND" device=""/>
-<part name="R1" library="freetronics" deviceset="RESISTOR" device="0603" value="10K 0603"/>
+<part name="R1" library="freetronics-master-v1.1" deviceset="RESISTOR" device="0603" value="10K 0603"/>
 <part name="F1" library="rcl" deviceset="L-EU" device="L1812" value="500mA PTC 1812"/>
-<part name="R2" library="freetronics" deviceset="RESISTOR" device="0603" value="1K 0603"/>
-<part name="R3" library="freetronics" deviceset="RESISTOR" device="0603" value="1K 0603"/>
+<part name="R2" library="freetronics-master-v1.1" deviceset="RESISTOR" device="0603" value="1K 0603"/>
+<part name="R3" library="freetronics-master-v1.1" deviceset="RESISTOR" device="0603" value="1K 0603"/>
 <part name="LED1" library="freetronics-master-v1" deviceset="LED" device="0603" value="RX/GRN"/>
 <part name="LED2" library="freetronics-master-v1" deviceset="LED" device="0603" value="TX/YEL"/>
 <part name="U$2" library="SparkFun" deviceset="5V" device=""/>
-<part name="R4" library="freetronics" deviceset="RESISTOR" device="0603" value="1K 0603"/>
-<part name="R5" library="freetronics" deviceset="RESISTOR" device="0603" value="1K 0603"/>
+<part name="R4" library="freetronics-master-v1.1" deviceset="RESISTOR" device="0603" value="1K 0603"/>
+<part name="R5" library="freetronics-master-v1.1" deviceset="RESISTOR" device="0603" value="1K 0603"/>
 <part name="Q2" library="freetronics" deviceset="MOSFET-NCHANNEL" device="SMD" value="2N7002"/>
 <part name="GND9" library="SparkFun" deviceset="GND" device=""/>
 <part name="LED3" library="freetronics-master-v1" deviceset="LED" device="0603" value="D13/RED"/>
-<part name="R7" library="freetronics" deviceset="RESISTOR" device="0603" value="1K 0603"/>
-<part name="C8" library="freetronics" deviceset="CAP" device="0603" value="100nF 0603"/>
+<part name="R7" library="freetronics-master-v1.1" deviceset="RESISTOR" device="0603" value="1K 0603"/>
+<part name="C8" library="freetronics-master-v1.1" deviceset="CAP" device="0603" value="100nF 0603"/>
 <part name="SJ1" library="freetronics-jon" deviceset="SJC" device="N" value="RESET-EN"/>
-<part name="C9" library="freetronics" deviceset="CAP" device="0603" value="100nF 0603"/>
+<part name="C9" library="freetronics-master-v1.1" deviceset="CAP" device="0603" value="100nF 0603"/>
 <part name="GND11" library="SparkFun" deviceset="GND" device=""/>
 <part name="P2" library="pinhead" deviceset="PINHD-2X3" device="" value="ICSP:MAIN"/>
 <part name="GND22" library="SparkFun" deviceset="GND" device=""/>
-<part name="R10" library="freetronics" deviceset="RESISTOR" device="0603" value="820R 0603"/>
+<part name="R10" library="freetronics-master-v1.1" deviceset="RESISTOR" device="0603" value="820R 0603"/>
 <part name="LED4" library="freetronics-master-v1" deviceset="LED" device="0603" value="3V3/BLUE"/>
 <part name="GND23" library="SparkFun" deviceset="GND" device=""/>
 <part name="U$5" library="freetronics" deviceset="FIDUCIAL" device="1X2.5"/>
 <part name="U$14" library="freetronics" deviceset="FIDUCIAL" device="1X2.5"/>
-<part name="C11" library="freetronics" deviceset="CAP" device="0603" value="100nF 0603"/>
-<part name="R11" library="freetronics" deviceset="RESISTOR" device="0603" value="27R 0603"/>
-<part name="R12" library="freetronics" deviceset="RESISTOR" device="0603" value="27R 0603"/>
-<part name="R6" library="freetronics" deviceset="RESISTOR" device="0603" value="1M 0603"/>
+<part name="C11" library="freetronics-master-v1.1" deviceset="CAP" device="0603" value="100nF 0603"/>
+<part name="R11" library="freetronics-master-v1.1" deviceset="RESISTOR" device="0603" value="27R 0603"/>
+<part name="R12" library="freetronics-master-v1.1" deviceset="RESISTOR" device="0603" value="27R 0603"/>
+<part name="R6" library="freetronics-master-v1.1" deviceset="RESISTOR" device="0603" value="1M 0603"/>
 <part name="C12" library="freetronics-jon" deviceset="C-EU" device="C0603" value="47pF 0603"/>
 <part name="C13" library="freetronics-jon" deviceset="C-EU" device="C0603" value="47pF 0603"/>
@@
 <part name="P+8" library="freetronics-original" deviceset="VCC" device=""/>
 <part name="P+7" library="freetronics-master-v1.1" deviceset="3V3" device=""/>
-<part name="R8" library="freetronics" deviceset="RESISTOR" device="0603" value="1K 0603"/>
-<part name="R9" library="freetronics" deviceset="RESISTOR" device="0603" value="1K 0603"/>
+<part name="R8" library="freetronics-master-v1.1" deviceset="RESISTOR" device="0603" value="1K 0603"/>
+<part name="R9" library="freetronics-master-v1.1" deviceset="RESISTOR" device="0603" value="1K 0603"/>
 <part name="IC3" library="freetronics-luke" deviceset="LTC4054" device=""/>
-<part name="R13" library="freetronics" deviceset="RESISTOR" device="0603" value="1K 0603"/>
-<part name="R14" library="freetronics" deviceset="RESISTOR" device="0603" value="1K 0603"/>
-<part name="C1" library="freetronics" deviceset="CAP" device="0603" value="1uF 0603"/>
-<part name="R15" library="freetronics" deviceset="RESISTOR" device="0603" value="10K 0603"/>
+<part name="R13" library="freetronics-master-v1.1" deviceset="RESISTOR" device="0603" value="1K 0603"/>
+<part name="R14" library="freetronics-master-v1.1" deviceset="RESISTOR" device="0603" value="1K 0603"/>
+<part name="C1" library="freetronics-master-v1.1" deviceset="CAP" device="0603" value="1uF 0603"/>
+<part name="R15" library="freetronics-master-v1.1" deviceset="RESISTOR" device="0603" value="10K 0603"/>
 <part name="LED5" library="freetronics-master-v1" deviceset="LED" device="0603" value="CHRG/ORANGE"/>
 <part name="LED6" library="freetronics-master-v1" deviceset="LED" device="0603" value="STBY/GREEN"/>
 <part name="Q1" library="freetronics-luke" deviceset="2N7002" device="" value="2N7002 SOT-23"/>
-<part name="R16" library="freetronics" deviceset="RESISTOR" device="0603" value="3K3 0603"/>
-<part name="R17" library="freetronics" deviceset="RESISTOR" device="0603" value="10K 0603"/>
+<part name="R16" library="freetronics-master-v1.1" deviceset="RESISTOR" device="0603" value="3K3 0603"/>
+<part name="R17" library="freetronics-master-v1.1" deviceset="RESISTOR" device="0603" value="10K 0603"/>
 <part name="SJ4" library="freetronics-jon" deviceset="SJC" device="N"/>
 <part name="SJ5" library="freetronics-jon" deviceset="SJC" device="N"/>
@@
 <part name="GND16" library="SparkFun" deviceset="GND" device=""/>
 <part name="IC4" library="freetronics-jon" deviceset="TEXAS_TPS770*" device="" technology="33" value="LP2985-33DBVR"/>
-<part name="C7" library="freetronics" deviceset="CAP" device="0603" value="1uF 0603"/>
+<part name="C7" library="freetronics-master-v1.1" deviceset="CAP" device="0603" value="1uF 0603"/>
 <part name="P+10" library="freetronics-original" deviceset="VCC" device=""/>
 <part name="P+11" library="freetronics-master-v1.1" deviceset="3V3" device=""/>
 <part name="GND8" library="SparkFun" deviceset="GND" device=""/>
 <part name="S4" library="freetronics-jon" deviceset="AUDIO-JACK-4POLE" device="" value="4UCON-18899"/>
-<part name="R18" library="freetronics" deviceset="RESISTOR" device="0603" value="10K 0603"/>
+<part name="R18" library="freetronics-master-v1.1" deviceset="RESISTOR" device="0603" value="10K 0603"/>
 <part name="GND7" library="SparkFun" deviceset="GND" device=""/>
 <part name="P+12" library="freetronics-original" deviceset="VCC" device=""/>
@@
 <part name="LED7" library="freetronics-master-v1" deviceset="LED" device="0603" value="5V/JADEGREEN"/>
 <part name="GND14" library="SparkFun" deviceset="GND" device=""/>
-<part name="R19" library="freetronics" deviceset="RESISTOR" device="0603" value="2K7 0603"/>
+<part name="R19" library="freetronics-master-v1.1" deviceset="RESISTOR" device="0603" value="2K7 0603"/>
 <part name="U$3" library="SparkFun" deviceset="5V" device=""/>
 <part name="SJ6" library="freetronics-master-v1.1" deviceset="SJ" device="" value="LINK"/>
